Commit message: [openrr-planner] Update sample model
This is to make it easy to how collision checking.

* large root body to make it easy to collide with arm
* large joint range for the same reason
* fix test for that change

File: openrr-planner/sample.urdf (robot description, URDF)
Before this commit: robot robo, 10 links, 9 joints
Links:
- link root: geometry collision box size=0.5 0.3 0.6; visual box size=0.5 0.3 0.6
Joints:
- joint l_shoulder_yaw: limit lower=-1.5 upper=1.5 effort=0 velocity=1.0 -> lower=-3 upper=3 effort=0 velocity=1.0
- joint l_wrist_yaw: limit lower=-1.5 upper=1.5 effort=0 velocity=1.0 -> lower=-3 upper=3 effort=0 velocity=1.0

Commit message: [openrr-planner] Change the sample robot model

File: openrr-planner/sample.urdf (robot description, URDF)
Before this commit: robot robo, 10 links, 9 joints
Links:
- removed link l_gripper1
- removed link l_gripper2
- removed link l_tool
- added link r_elbow1; collision box size=0.1 0.1 0.2; visual box size=0.1 0.1 0.2
- added link r_shoulder1; collision box size=0.1 0.1 0.1; visual box size=0.1 0.1 0.1
- added link r_shoulder2; collision box size=0.1 0.1 0.1; visual box size=0.1 0.1 0.1
- added link r_shoulder3; collision box size=0.1 0.1 0.2; visual box size=0.1 0.1 0.2
- added link r_wrist1; collision cylinder length=0.2 radius=0.1; visual cylinder length=0.2 radius=0.1
- added link r_wrist2; collision box size=0.05 0.08 0.15; visual box size=0.05 0.08 0.15
- link l_elbow1: geometry collision box size=0.1 0.1 0.2; visual box size=0.1 0.1 0.2
- link l_shoulder3: geometry collision box size=0.1 0.1 0.2; visual box size=0.1 0.1 0.2
- link l_wrist1: geometry collision cylinder length=0.2 radius=0.1; visual cylinder length=0.2 radius=0.1
- link l_wrist2: geometry collision box size=0.05 0.08 0.15; visual box size=0.05 0.08 0.15
- link root: geometry collision box size=0.2 0.2 0.4; collision sphere radius=0.2
Joints:
- removed joint l_gripper_linear1
- removed joint l_gripper_linear2
- removed joint l_tool_fixed
- added joint r_elbow_pitch: type revolute, parent r_shoulder3, child r_elbow1, origin xyz=0.0 0.0 -0.2, axis 0 1 0, limit lower=-2 upper=1.0 effort=0 velocity=1.0
- added joint r_shoulder_pitch: type revolute, parent r_shoulder1, child r_shoulder2, origin xyz=0.0 -0.1 0.0, axis 0 1 0, limit lower=-1 upper=1.0 effort=0 velocity=1.0
- added joint r_shoulder_roll: type revolute, parent r_shoulder2, child r_shoulder3, origin xyz=0.0 -0.1 0.0, axis 1 0 0, limit lower=-2 upper=1.0 effort=0 velocity=1.0
- added joint r_shoulder_yaw: type revolute, parent root, child r_shoulder1, origin xyz=0.0 -0.2 0.2, axis 0 0 1, limit lower=-1 upper=1.0 effort=0 velocity=1.0
- added joint r_wrist_pitch: type revolute, parent r_wrist1, child r_wrist2, origin xyz=0.0 0.0 -0.2, axis 0 1 0, limit lower=-2 upper=1.0 effort=0 velocity=1.0
- added joint r_wrist_yaw: type revolute, parent r_elbow1, child r_wrist1, origin xyz=0.0 0.0 -0.2, axis 0 0 1, limit lower=-2 upper=1.0 effort=0 velocity=1.0
- joint l_elbow_pitch: limit lower=-2.0 upper=1.5 effort=0 velocity=1.0 -> lower=-2 upper=1.0 effort=0 velocity=1.0; origin xyz=0.3 0.0 0.0 -> xyz=0.0 0.0 -0.2
- joint l_shoulder_pitch: limit lower=-2.0 upper=1.5 effort=0 velocity=1.0 -> lower=-1 upper=1.0 effort=0 velocity=1.0
- joint l_shoulder_roll: limit lower=-1.5 upper=2.0 effort=0 velocity=1.0 -> lower=-2 upper=1.0 effort=0 velocity=1.0
- joint l_shoulder_yaw: limit lower=-3 upper=3 effort=0 velocity=1.0 -> lower=-1 upper=1.0 effort=0 velocity=1.0; origin xyz=0.0 0.2 0.5 -> xyz=0.0 0.2 0.2
- joint l_wrist_pitch: limit lower=-2 upper=2.0 effort=0 velocity=1.0 -> lower=-2 upper=1.0 effort=0 velocity=1.0; origin xyz=0.15 0.0 0.0 -> xyz=0.0 0.0 -0.2
- joint l_wrist_yaw: limit lower=-3 upper=3 effort=0 velocity=1.0 -> lower=-2 upper=1.0 effort=0 velocity=1.0; origin xyz=0.25 0.0 0.0 -> xyz=0.0 0.0 -0.2

Commit message: [openrr-planner] Change the sample robot model

File: openrr-planner/sample.urdf (robot description, URDF)
Before this commit: robot robo, 10 links, 9 joints
Links:
- added link r_elbow1; collision box size=0.25 0.05 0.1; visual box size=0.25 0.05 0.1
- added link r_gripper1; collision cylinder length=0.15 radius=0.02; visual cylinder length=0.15 radius=0.02
- added link r_gripper2; collision cylinder length=0.15 radius=0.02; visual cylinder length=0.15 radius=0.02
- added link r_shoulder1; collision box size=0.1 0.1 0.1; visual box size=0.1 0.1 0.1
- added link r_shoulder2; collision box size=0.1 0.1 0.1; visual box size=0.1 0.1 0.1
- added link r_shoulder3; collision box size=0.25 0.1 0.15; visual box size=0.25 0.1 0.15
- added link r_tool; visual box size=0.01 0.01 0.01
- added link r_wrist1; collision box size=0.25 0.15 0.1; visual box size=0.25 0.15 0.1
- added link r_wrist2; collision box size=0.1 0.08 0.05; visual box size=0.1 0.08 0.05
Joints:
- added joint r_elbow_pitch: type revolute, parent r_shoulder3, child r_elbow1, origin xyz=0.3 0.0 0.0, axis 0 1 0, limit lower=-2.0 upper=1.5 effort=0 velocity=1.0
- added joint r_gripper_linear1: type prismatic, parent r_wrist2, child r_gripper1, origin xyz=0.15 -0.05 0.0 rpy=0 0 1.57, axis 1 0 0, limit lower=-0.05 upper=0.05 effort=0 velocity=1.0
- added joint r_gripper_linear2: type prismatic, parent r_wrist2, child r_gripper2, origin xyz=0.15 0.05 0.0 rpy=0 0 1.57, axis 1 0 0, limit lower=-0.05 upper=0.05 effort=0 velocity=1.0, mimic joint=r_gripper_linear1 multiplier=-1.0
- added joint r_shoulder_pitch: type revolute, parent r_shoulder1, child r_shoulder2, origin xyz=0.0 -0.1 0.0, axis 0 1 0, limit lower=-2.0 upper=1.5 effort=0 velocity=1.0
- added joint r_shoulder_roll: type revolute, parent r_shoulder2, child r_shoulder3, origin xyz=0.0 -0.1 0.0, axis 1 0 0, limit lower=-1.5 upper=2.0 effort=0 velocity=1.0
- added joint r_shoulder_yaw: type revolute, parent root, child r_shoulder1, origin xyz=0.0 -0.2 0.5, axis 0 0 1, limit lower=-3 upper=3 effort=0 velocity=1.0
- added joint r_tool_fixed: type fixed, parent r_wrist2, child r_tool, origin xyz=0.2 0.0 0.0
- added joint r_wrist_pitch: type revolute, parent r_wrist1, child r_wrist2, origin xyz=0.15 0.0 0.0, axis 0 1 0, limit lower=-2 upper=2.0 effort=0 velocity=1.0
- added joint r_wrist_yaw: type revolute, parent r_elbow1, child r_wrist1, origin xyz=0.25 0.0 0.0, axis 0 0 1, limit lower=-3 upper=3 effort=0 velocity=1.0
